File: hand.brd (EAGLE design)
At the start: 299.4 x 150.4 mm, 31 parts, among them IC1 74HC366N, IC2 74HC366N, IC3 74HC366N, IC4 74HC366N

Commit message: Add files via upload
Parts:
- moved C-OR 9.71 mm to (105.1, 80.0)
- moved IC-OR 9.69 mm to (92.8, 75.9), turned to 162 degrees
Routing:
- net LED1-CA: track 46.0 -> 0.00 mm
- net LED6-AN: track 46.0 -> 0.00 mm
- net LED1-AN: track 45.6 -> 0.00 mm
- net LED6-CA: track 45.6 -> 0.00 mm
- net LED9-AN: track 38.7 -> 0.00 mm
- net LED9-CA: track 38.3 -> 0.00 mm
- net LED2-CA: track 28.8 -> 0.00 mm
- net LED5-AN: track 28.8 -> 0.00 mm
- net LED5-CA: track 28.6 -> 0.00 mm
- net LED2-AN: track 28.6 -> 0.00 mm
- net LED7-CA: track 24.0 -> 0.00 mm
- net LED10-AN: track 24.0 -> 0.00 mm
- net LED10-CA: track 23.7 -> 0.00 mm
- net LED7-AN: track 23.7 -> 0.00 mm
- net LED8-AN: track 21.5 -> 0.00 mm
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